Commit message: modify: collision model
Nisopa_kerb_ramp

File: urdf/obstacles/Nisopa_Kerb_Ramp.urdf.xacro (robot description, xacro)
@@ -2,4 +2,5 @@
 <robot xmlns:xacro="http://www.ros.org/wiki/xacro">
   <xacro:macro name="Nisopa_Kerb_Ramp" params="handle parent position orientation">
+  <!-- visual mesh -->
   <joint name="Nisopa_Kerb_Ramp_${handle}_joint" type="fixed">
     <origin xyz="${position}" rpy="${orientation}"/>
@@ -28,7 +29,31 @@
           name="">
           <color
-            rgba="0.40 0.39 0.43 1" />
+            rgba="1 0 0 1" />
         </material>
       </visual>
+    </link>
+    <gazebo reference="Nisopa_Kerb_Ramp_${handle}">
+      <material>Gazebo/DarkGrey</material>
+    </gazebo>
+  <!-- collision links -->
+  <joint name="Nisopa_Kerb_Ramp_${handle}_collision_joint_1" type="fixed">
+    <origin xyz="-2.3000e-02 0 -7.1000e-02"
+            rpy="0 0 0"/>
+    <parent link="Nisopa_Kerb_Ramp_${handle}"/>
+    <child link="Nisopa_Kerb_Ramp_${handle}_collision_1"/>
+  </joint>
+  <link
+      name="Nisopa_Kerb_Ramp_${handle}_collision_1">
+      <inertial>
+        <origin xyz="0 0 0" rpy="0 0 0"/>
+        <mass value="1.663e+00"/>
+          <inertia
+        ixx="+1.881e-02"
+        ixy="0.0"
+        ixz="0.0"
+        iyz="+1.022e-02"
+        iyy="0.0"
+        izz="+2.901e-02" />
+      </inertial>
       <collision>
         <origin
@@ -36,12 +61,79 @@
           rpy="0 0 0" />
         <geometry>
-          <mesh
-            filename="package://ICRA2023_Quadruped_Competition/meshes/Nisopa_Kerb_Ramp.stl" />
+          <box size="3.5000e-01 4.7500e-01 1.0000e-02" />
         </geometry>
+        <material
+          name="">
+          <color
+            rgba="1 0 0 1" />
+        </material>
       </collision>
     </link>
-    <gazebo reference="Nisopa_Kerb_Ramp_${handle}">
-      <material>Gazebo/DarkGrey</material>
-    </gazebo>
+  <joint name="Nisopa_Kerb_Ramp_${handle}_collision_joint_2" type="fixed">
+    <origin xyz="-1.9400e-01  0  +9.9994e-04"
+            rpy="0 0 0"/>
+    <parent link="Nisopa_Kerb_Ramp_${handle}"/>
+    <child link="Nisopa_Kerb_Ramp_${handle}_collision_2"/>
+  </joint>
+  <link
+      name="Nisopa_Kerb_Ramp_${handle}_collision_2">
+      <inertial>
+        <origin xyz="0 0 0" rpy="0 0 0"/>
+        <mass value="6.175e-01"/>
+          <inertia
+        ixx="+2.021e-02"
+        ixy="0.0"
+        ixz="0.0"
+        iyz="+1.417e-03"
+        iyy="0.0"
+        izz="+1.881e-02" />
+      </inertial>
+      <collision>
+        <origin
+          xyz="0 0 0"
+          rpy="0 0 0" />
+        <geometry>
+          <box size="1.0000e-02 4.7500e-01 1.3000e-01" />
+        </geometry>
+        <material
+          name="">
+          <color
+            rgba="1 0 0 1" />
+        </material>
+      </collision>
+    </link>
+  <joint name="Nisopa_Kerb_Ramp_${handle}_collision_joint_3" type="fixed">
+    <origin xyz="-1.9488e-03  0  -2.1460e-03"
+            rpy="0 0.3577925 0"/>
+    <parent link="Nisopa_Kerb_Ramp_${handle}"/>
+    <child link="Nisopa_Kerb_Ramp_${handle}_collision_3"/>
+  </joint>
+  <link
+      name="Nisopa_Kerb_Ramp_${handle}_collision_3">
+      <inertial>
+        <origin xyz="0 0 0" rpy="0 0 0"/>
+        <mass value="1.995e+00"/>
+          <inertia
+        ixx="+2.061e-02"
+        ixy="0.0"
+        ixz="+4.819e-03"
+        iyz="+1.471e-02"
+        iyy="0.0"
+        izz="3.170e-02" />
+      </inertial>
+      <collision>
+        <origin
+          xyz="0 0 0"
+          rpy="0 0 0" />
+        <geometry>
+          <box size="4.2000e-01 4.7500e-01 1.0000e-02" />
+        </geometry>
+        <material
+          name="">
+          <color
+            rgba="1 0 0 1" />
+        </material>
+      </collision>
+    </link>
   </xacro:macro>
 </robot>
