Commit message: modify: collision model
New_600x400_2way

File: urdf/obstacles/New_600x400_2way_Wooden_Pallet.urdf.xacro (robot description, xacro)
@@ -2,4 +2,5 @@
 <robot xmlns:xacro="http://www.ros.org/wiki/xacro">
   <xacro:macro name="New_600x400_2way_Wooden_Pallet" params="handle parent position orientation">
+  <!-- visual mesh-->
   <joint name="New_600x400_2way_Wooden_Pallet_${handle}_joint" type="fixed">
     <origin xyz="${position}" rpy="${orientation}"/>
@@ -7,14 +8,15 @@
     <child link="New_600x400_2way_Wooden_Pallet_${handle}"/>
   </joint>
-    <link
-      name="New_600x400_2way_Wooden_Pallet_${handle}">
-      <inertial>
-        <origin xyz="0 0 0.5" rpy="0 0 0"/>
-        <mass value="1"/>
+  <link
+    name="New_600x400_2way_Wooden_Pallet_${handle}">
+      <!--
+      <inertial>
+        <origin xyz="0 0 0" rpy="0 0 0"/>
+        <mass value="2.385e+01"/>
         <inertia
-      ixx="1.0" ixy="0.0" ixz="0.0"
-      iyy="1.0" iyz="0.0"
-      izz="1.0"/>
-      </inertial>
+        ixx="+1.051e-02" ixy="0.0" ixz="-7.090e-09"
+        iyx="0.0" iyy="+4.020e-02" iyz="0.0"
+        izx="-7.090e-09" izy="0.0" izz="+4.897e-02"/>
+      </inertial>-->
       <visual>
         <origin
@@ -28,18 +30,225 @@
           name="">
           <color
-            rgba="0.22 0.76 0.94 1" />
-          <texture filename="package://ICRA2023_Quadruped_Competition/textures/wooden.jpg" />
+            rgba="1 0 0 1" />
         </material>
       </visual>
-      <collision>
-        <origin
-          xyz="0 0 0"
-          rpy="0 0 0" />
-        <geometry>
-          <mesh
-            filename="package://ICRA2023_Quadruped_Competition/meshes/New_600x400_2way_Wooden_Pallet.dae" />
-        </geometry>
-      </collision>
-    </link>
+    </link>
+  <!-- collision links -->
+  <joint name="New_600x400_2way_Wooden_Pallet_${handle}_collision_joint_1" type="fixed">
+    <origin xyz="+2.8100e-01 +0.0000e+00 -7.9997e-03"
+            rpy="0 0 1.5708"/>
+    <parent link="New_600x400_2way_Wooden_Pallet_${handle}"/>
+    <child link="New_600x400_2way_Wooden_Pallet_${handle}_collision_1"/>
+  </joint>
+  <link
+      name="New_600x400_2way_Wooden_Pallet_${handle}_collision_1">
+      <inertial>
+        <origin xyz="0 0 0" rpy="0 0 0"/>
+        <mass value="1.520e+00"/>
+          <inertia
+        ixx="+1.417e-02"
+        ixy="+1.103e-07"
+        ixz="+0.000e+00"
+        iyz="+1.103e-07"
+        iyy="+9.537e-04"
+        izz="+1.345e-02" />
+      </inertial>
+      <collision>
+        <origin
+          xyz="0 0 0"
+          rpy="0 0 0" />
+        <geometry>
+          <box size="4.0000e-01 3.8000e-02 1.0000e-01" />
+        </geometry>
+        <material
+          name="">
+          <color
+            rgba="1 0 0 1" />
+        </material>
+      </collision>
+    </link>
+    <gazebo reference="New_600x400_2way_Wooden_Pallet_${handle}_collision_1">
+      <selfCollide>false</selfCollide>
+    </gazebo>
+  <joint name="New_600x400_2way_Wooden_Pallet_${handle}_collision_joint_2" type="fixed">
+    <origin xyz="-2.8100e-01 +0.0000e+00 -7.9997e-03"
+            rpy="0 0 1.5708"/>
+    <parent link="New_600x400_2way_Wooden_Pallet_${handle}"/>
+    <child link="New_600x400_2way_Wooden_Pallet_${handle}_collision_2"/>
+  </joint>
+  <link
+      name="New_600x400_2way_Wooden_Pallet_${handle}_collision_2">
+      <inertial>
+        <origin xyz="0 0 0" rpy="0 0 0"/>
+        <mass value="1.520e+00"/>
+          <inertia
+        ixx="+1.417e-02"
+        ixy="+1.103e-07"
+        ixz="+0.000e+00"
+        iyz="+1.103e-07"
+        iyy="+9.537e-04"
+        izz="+1.345e-02" />
+      </inertial>
+      <collision>
+        <origin
+          xyz="0 0 0"
+          rpy="0 0 0" />
+        <geometry>
+          <box size="4.0000e-01 3.8000e-02 1.0000e-01" />
+        </geometry>
+        <material
+          name="">
+          <color
+            rgba="1 0 0 1" />
+        </material>
+      </collision>
+    </link>
+    <gazebo reference="New_600x400_2way_Wooden_Pallet_${handle}_collision_2">
+      <selfCollide>false</selfCollide>
+    </gazebo>
+  <joint name="New_600x400_2way_Wooden_Pallet_${handle}_collision_joint_3" type="fixed">
+    <origin xyz="+0.0000e+00 +1.6250e-01 +5.0000e-02"
+            rpy="0 1.5708 1.5708"/>
+    <parent link="New_600x400_2way_Wooden_Pallet_${handle}"/>
+    <child link="New_600x400_2way_Wooden_Pallet_${handle}_collision_3"/>
+  </joint>
+  <link
+      name="New_600x400_2way_Wooden_Pallet_${handle}_collision_3">
+      <inertial>
+        <origin xyz="0 0 0" rpy="0 0 0"/>
+        <mass value="7.200e-01"/>
+          <inertia
+        ixx="+4.901e-04"
+        ixy="0.0"
+        ixz="+0.000e+00"
+        iyz="+3.002e-02"
+        iyy="0.0"
+        izz="+3.047e-02" />
+      </inertial>
+      <collision>
+        <origin
+          xyz="0 0 0"
+          rpy="0 0 0" />
+        <geometry>
+          <box size="1.6000e-02 6.0000e-01 7.5000e-02" />
+        </geometry>
+        <material
+          name="">
+          <color
+            rgba="1 0 0 1" />
+        </material>
+      </collision>
+    </link>
+    <gazebo reference="New_600x400_2way_Wooden_Pallet_${handle}_collision_3">
+      <selfCollide>false</selfCollide>
+    </gazebo>
+  <joint name="New_600x400_2way_Wooden_Pallet_${handle}_collision_joint_4" type="fixed">
+    <origin xyz="+0.0000e+00 +5.4167e-02 +5.0000e-02"
+            rpy="0 1.5708 1.5708"/>
+    <parent link="New_600x400_2way_Wooden_Pallet_${handle}"/>
+    <child link="New_600x400_2way_Wooden_Pallet_${handle}_collision_4"/>
+  </joint>
+  <link
+      name="New_600x400_2way_Wooden_Pallet_${handle}_collision_4">
+      <inertial>
+        <origin xyz="0 0 0" rpy="0 0 0"/>
+        <mass value="7.200e-01"/>
+          <inertia
+        ixx="+4.901e-04"
+        ixy="0.0"
+        ixz="+0.000e+00"
+        iyz="+3.002e-02"
+        iyy="0.0"
+        izz="+3.047e-02" />
+      </inertial>
+      <collision>
+        <origin
+          xyz="0 0 0"
+          rpy="0 0 0" />
+        <geometry>
+          <box size="1.6000e-02 6.0000e-01 7.5000e-02" />
+        </geometry>
+        <material
+          name="">
+          <color
+            rgba="1 0 0 1" />
+        </material>
+      </collision>
+    </link>
+    <gazebo reference="New_600x400_2way_Wooden_Pallet_${handle}_collision_4">
+      <selfCollide>false</selfCollide>
+    </gazebo>
+  <joint name="New_600x400_2way_Wooden_Pallet_${handle}_collision_joint_5" type="fixed">
+    <origin xyz="+0.0000e+00 -5.4167e-02 +5.0000e-02"
+            rpy="0 1.5708 1.5708"/>
+    <parent link="New_600x400_2way_Wooden_Pallet_${handle}"/>
+    <child link="New_600x400_2way_Wooden_Pallet_${handle}_collision_5"/>
+  </joint>
+  <link
+      name="New_600x400_2way_Wooden_Pallet_${handle}_collision_5">
+      <inertial>
+        <origin xyz="0 0 0" rpy="0 0 0"/>
+        <mass value="7.200e-01"/>
+          <inertia
+        ixx="+4.901e-04"
+        ixy="0.0"
+        ixz="+0.000e+00"
+        iyz="+3.002e-02"
+        iyy="0.0"
+        izz="+3.047e-02" />
+      </inertial>
+      <collision>
+        <origin
+          xyz="0 0 0"
+          rpy="0 0 0" />
+        <geometry>
+          <box size="1.6000e-02 6.0000e-01 7.5000e-02" />
+        </geometry>
+        <material
+          name="">
+          <color
+            rgba="1 0 0 1" />
+        </material>
+      </collision>
+    </link>
+    <gazebo reference="New_600x400_2way_Wooden_Pallet_${handle}_collision_5">
+      <selfCollide>false</selfCollide>
+    </gazebo>
+  <joint name="New_600x400_2way_Wooden_Pallet_${handle}_collision_joint_6" type="fixed">
+    <origin xyz="+0.0000e+00 -1.6250e-01 +5.0000e-02"
+            rpy="0 1.5708  1.5708"/>
+    <parent link="New_600x400_2way_Wooden_Pallet_${handle}"/>
+    <child link="New_600x400_2way_Wooden_Pallet_${handle}_collision_6"/>
+  </joint>
+  <link
+      name="New_600x400_2way_Wooden_Pallet_${handle}_collision_6">
+       <inertial>
+        <origin xyz="0 0 0" rpy="0 0 0"/>
+        <mass value="7.200e-01"/>
+          <inertia
+        ixx="+4.901e-04"
+        ixy="0.0"
+        ixz="+0.000e+00"
+        iyz="+3.002e-02"
+        iyy="0.0"
+        izz="+3.047e-02" />
+      </inertial>
+      <collision>
+        <origin
+          xyz="0 0 0"
+          rpy="0 0 0" />
+        <geometry>
+          <box size="1.6000e-02 6.0000e-01 7.5000e-02" />
+        </geometry>
+        <material
+          name="">
+          <color
+            rgba="1 0 0 1" />
+        </material>
+      </collision>
+    </link>
+    <gazebo reference="New_600x400_2way_Wooden_Pallet_${handle}_collision_6">
+      <selfCollide>false</selfCollide>
+    </gazebo>
   </xacro:macro>
 </robot>

File: urdf/obstacles/Plywood_wall.urdf.xacro (robot description, xacro)
@@ -28,6 +28,5 @@
           name="">
           <color
-            rgba="0.22 0.76 0.94 1" />
-          <texture filename="package://ICRA2023_Quadruped_Competition/textures/wooden.jpg" />
+            rgba="1 0 0 1" />
         </material>
       </visual>
@@ -37,6 +36,5 @@
           rpy="0 0 0" />
         <geometry>
-          <mesh
-            filename="package://ICRA2023_Quadruped_Competition/meshes/Plywood_wall.dae" />
+          <box size="6.1000e-01 1.2000e-02 5.9500e-01" />
         </geometry>
       </collision>

Commit message: modify: collision model
New_EURO_EPAL_pallet

File: urdf/obstacles/New_600x400_2way_Wooden_Pallet.urdf.xacro (robot description, xacro)
@@ -68,7 +68,4 @@
       </collision>
     </link>
-    <gazebo reference="New_600x400_2way_Wooden_Pallet_${handle}_collision_1">
-      <selfCollide>false</selfCollide>
-    </gazebo>
   <joint name="New_600x400_2way_Wooden_Pallet_${handle}_collision_joint_2" type="fixed">
     <origin xyz="-2.8100e-01 +0.0000e+00 -7.9997e-03"
@@ -104,7 +101,4 @@
       </collision>
     </link>
-    <gazebo reference="New_600x400_2way_Wooden_Pallet_${handle}_collision_2">
-      <selfCollide>false</selfCollide>
-    </gazebo>
   <joint name="New_600x400_2way_Wooden_Pallet_${handle}_collision_joint_3" type="fixed">
     <origin xyz="+0.0000e+00 +1.6250e-01 +5.0000e-02"
@@ -140,7 +134,4 @@
       </collision>
     </link>
-    <gazebo reference="New_600x400_2way_Wooden_Pallet_${handle}_collision_3">
-      <selfCollide>false</selfCollide>
-    </gazebo>
   <joint name="New_600x400_2way_Wooden_Pallet_${handle}_collision_joint_4" type="fixed">
     <origin xyz="+0.0000e+00 +5.4167e-02 +5.0000e-02"
@@ -176,7 +167,4 @@
       </collision>
     </link>
-    <gazebo reference="New_600x400_2way_Wooden_Pallet_${handle}_collision_4">
-      <selfCollide>false</selfCollide>
-    </gazebo>
   <joint name="New_600x400_2way_Wooden_Pallet_${handle}_collision_joint_5" type="fixed">
     <origin xyz="+0.0000e+00 -5.4167e-02 +5.0000e-02"
@@ -212,7 +200,4 @@
       </collision>
     </link>
-    <gazebo reference="New_600x400_2way_Wooden_Pallet_${handle}_collision_5">
-      <selfCollide>false</selfCollide>
-    </gazebo>
   <joint name="New_600x400_2way_Wooden_Pallet_${handle}_collision_joint_6" type="fixed">
     <origin xyz="+0.0000e+00 -1.6250e-01 +5.0000e-02"
@@ -248,7 +233,4 @@
       </collision>
     </link>
-    <gazebo reference="New_600x400_2way_Wooden_Pallet_${handle}_collision_6">
-      <selfCollide>false</selfCollide>
-    </gazebo>
   </xacro:macro>
 </robot>

File: urdf/obstacles/New_EURO_EPAL_Pallet.urdf.xacro (robot description, xacro)
@@ -2,4 +2,5 @@
 <robot xmlns:xacro="http://www.ros.org/wiki/xacro">
   <xacro:macro name="New_EURO_EPAL_Pallet" params="handle parent position orientation">
+  <!-- visual mesh -->
   <joint name="New_EURO_EPAL_Pallet_${handle}_joint" type="fixed">
     <origin xyz="${position}" rpy="${orientation}"/>
@@ -7,29 +8,42 @@
     <child link="New_EURO_EPAL_Pallet_${handle}"/>
   </joint>
-    <link
-      name="New_EURO_EPAL_Pallet_${handle}">
+  <link
+    name="New_EURO_EPAL_Pallet_${handle}">
+    <visual>
+      <origin
+        xyz="0 0 0"
+        rpy="0 0 0" />
+      <geometry>
+        <mesh
+          filename="package://ICRA2023_Quadruped_Competition/meshes/New_EURO_EPAL_Pallet.dae"/>
+      </geometry>
+      <material
+        name="">
+        <color
+          rgba="0.22 0.76 0.94 1" />
+        <texture filename="package://ICRA2023_Quadruped_Competition/textures/wooden.jpg" />
+      </material>
+    </visual>
+  </link>
+  <!-- collision links -->
+  <joint name="New_EURO_EPAL_Pallet_${handle}_collision_joint_1" type="fixed">
+    <origin xyz="0 0 +6.1000e-02"
+            rpy="0 0 0"/>
+    <parent link="New_EURO_EPAL_Pallet_${handle}"/>
+    <child link="New_EURO_EPAL_Pallet_${handle}_collision_1"/>
+  </joint>
+  <link
+      name="New_EURO_EPAL_Pallet_${handle}_collision_1">
       <inertial>
-        <origin xyz="0 0 0.5" rpy="0 0 0"/>
-        <mass value="1"/>
-        <inertia
-      ixx="1.0" ixy="0.0" ixz="0.0"
-      iyy="1.0" iyz="0.0"
-      izz="1.0"/>
+        <origin xyz="0 0 0" rpy="0 0 0"/>
+        <mass value="3.828e+00"/>
+          <inertia
+        ixx="+1.200e-01"
+        ixy="+6.414e-06"
+        ixz="+3.621e-11"
+        iyz="+1.792e-03"
+        iyy="-2.528e-09"
+        izz="+1.218e-01" />
       </inertial>
-      <visual>
-        <origin
-          xyz="0 0 0"
-          rpy="0 0 0" />
-        <geometry>
-          <mesh
-            filename="package://ICRA2023_Quadruped_Competition/meshes/New_EURO_EPAL_Pallet.dae"/>
-        </geometry>
-        <material
-          name="">
-          <color
-            rgba="0.22 0.76 0.94 1" />
-          <texture filename="package://ICRA2023_Quadruped_Competition/textures/wooden.jpg" />
-        </material>
-      </visual>
       <collision>
         <origin
@@ -37,7 +51,143 @@
           rpy="0 0 0" />
         <geometry>
-          <mesh
-            filename="package://ICRA2023_Quadruped_Competition/meshes/New_EURO_EPAL_Pallet.dae" />
+          <box size="1.2000e+00  1.4500e-01  2.2000e-02" />
         </geometry>
+        <material
+          name="">
+          <color
+            rgba="1 0 0 1" />
+        </material>
+      </collision>
+    </link>
+  <joint name="New_EURO_EPAL_Pallet_${handle}_collision_joint_2" type="fixed">
+    <origin xyz="0 3.3000e-01 +6.1000e-02"
+            rpy="0 0 0"/>
+    <parent link="New_EURO_EPAL_Pallet_${handle}"/>
+    <child link="New_EURO_EPAL_Pallet_${handle}_collision_2"/>
+  </joint>
+  <link
+      name="New_EURO_EPAL_Pallet_${handle}_collision_2">
+      <inertial>
+        <origin xyz="0 0 0" rpy="0 0 0"/>
+        <mass value="3.828e+00"/>
+          <inertia
+        ixx="+1.200e-01"
+        ixy="+6.414e-06"
+        ixz="+3.621e-11"
+        iyz="+1.792e-03"
+        iyy="-2.528e-09"
+        izz="+1.218e-01" />
+      </inertial>
+      <collision>
+        <origin
+          xyz="0 0 0"
+          rpy="0 0 0" />
+        <geometry>
+          <box size="1.2000e+00  1.4500e-01  2.2000e-02" />
+        </geometry>
+        <material
+          name="">
+          <color
+            rgba="1 0 0 1" />
+        </material>
+      </collision>
+    </link>
+  <joint name="New_EURO_EPAL_Pallet_${handle}_collision_joint_3" type="fixed">
+    <origin xyz="0 -3.3000e-01 +6.1000e-02"
+            rpy="0 0 0"/>
+    <parent link="New_EURO_EPAL_Pallet_${handle}"/>
+    <child link="New_EURO_EPAL_Pallet_${handle}_collision_3"/>
+  </joint>
+  <link
+      name="New_EURO_EPAL_Pallet_${handle}_collision_3">
+      <inertial>
+        <origin xyz="0 0 0" rpy="0 0 0"/>
+        <mass value="3.828e+00"/>
+          <inertia
+        ixx="+1.200e-01"
+        ixy="+6.414e-06"
+        ixz="+3.621e-11"
+        iyz="+1.792e-03"
+        iyy="-2.528e-09"
+        izz="+1.218e-01" />
+      </inertial>
+      <collision>
+        <origin
+          xyz="0 0 0"
+          rpy="0 0 0" />
+        <geometry>
+          <box size="1.2000e+00  1.4500e-01  2.2000e-02" />
+        </geometry>
+        <material
+          name="">
+          <color
+            rgba="1 0 0 1" />
+        </material>
+      </collision>
+    </link>
+  <joint name="New_EURO_EPAL_Pallet_${handle}_collision_joint_4" type="fixed">
+    <origin xyz="0 1.6200e-01 +6.1000e-02"
+            rpy="0 0 0"/>
+    <parent link="New_EURO_EPAL_Pallet_${handle}"/>
+    <child link="New_EURO_EPAL_Pallet_${handle}_collision_4"/>
+  </joint>
+  <link
+      name="New_EURO_EPAL_Pallet_${handle}_collision_4">
+      <inertial>
+        <origin xyz="0 0 0" rpy="0 0 0"/>
+        <mass value="2.640e+00"/>
+          <inertia
+        ixx="+1.200e-01"
+        ixy="+3.651e-06"
+        ixz="-6.119e-18"
+        iyz="+8.737e-04"
+        iyy="-1.153e-14"
+        izz="+1.208e-01"/>
+      </inertial>
+      <collision>
+        <origin
+          xyz="0 0 0"
+          rpy="0 0 0" />
+        <geometry>
+          <box size="1.2000e+00  1.0000e-01  2.2000e-02" />
+        </geometry>
+        <material
+          name="">
+          <color
+            rgba="1 0 0 1" />
+        </material>
+      </collision>
+    </link>
+  <joint name="New_EURO_EPAL_Pallet_${handle}_collision_joint_5" type="fixed">
+    <origin xyz="0 -1.6200e-01 +6.1000e-02"
+            rpy="0 0 0"/>
+    <parent link="New_EURO_EPAL_Pallet_${handle}"/>
+    <child link="New_EURO_EPAL_Pallet_${handle}_collision_5"/>
+  </joint>
+  <link
+      name="New_EURO_EPAL_Pallet_${handle}_collision_5">
+      <inertial>
+        <origin xyz="0 0 0" rpy="0 0 0"/>
+        <mass value="3.828e+00"/>
+          <inertia
+        ixx="+1.200e-01"
+        ixy="+6.414e-06"
+        ixz="+3.621e-11"
+        iyz="+1.792e-03"
+        iyy="-2.528e-09"
+        izz="+1.218e-01" />
+      </inertial>
+      <collision>
+        <origin
+          xyz="0 0 0"
+          rpy="0 0 0" />
+        <geometry>
+          <box size="1.2000e+00  1.0000e-01  2.2000e-02" />
+        </geometry>
+        <material
+          name="">
+          <color
+            rgba="1 0 0 1" />
+        </material>
       </collision>
     </link>

Commit message: update: obstacles

File: urdf/obstacles/New_600x400_2way_Wooden_Pallet.urdf.xacro (robot description, xacro)
@@ -222,4 +222,7 @@
       </collision>
     </link>
+    <gazebo reference="New_600x400_2way_Wooden_Pallet_${handle}">
+      <material>Gazebo/Wood</material>
+    </gazebo>
   </xacro:macro>
 </robot>

File: urdf/obstacles/New_EURO_EPAL_Pallet.urdf.xacro (robot description, xacro)
@@ -189,4 +189,7 @@
       </collision>
     </link>
+    <gazebo reference="New_EURO_EPAL_Pallet_${handle}">
+      <material>Gazebo/Wood</material>
+    </gazebo>
   </xacro:macro>
 </robot>

File: urdf/obstacles/Plywood_16mm_sheet.urdf.xacro (robot description, xacro)
@@ -39,4 +39,7 @@
       </collision>
     </link>
+    <gazebo reference="Plywood_16mm_sheet_${handle}">
+      <material>Gazebo/Wood</material>
+    </gazebo>
   </xacro:macro>
 </robot>

File: urdf/obstacles/Plywood_3mm_sheet.urdf.xacro (robot description, xacro)
@@ -39,4 +39,7 @@
       </collision>
     </link>
+    <gazebo reference="Plywood_3mm_sheet_${handle}">
+      <material>Gazebo/Wood</material>
+    </gazebo>
   </xacro:macro>
 </robot>

File: urdf/obstacles/Plywood_wall.urdf.xacro (robot description, xacro)
@@ -38,4 +38,7 @@
       </collision>
     </link>
+    <gazebo reference="Plywood_wall_${handle}">
+      <material>Gazebo/Wood</material>
+    </gazebo>
   </xacro:macro>
 </robot>

File: urdf/obstacles/solid_wood_block.urdf.xacro (robot description, xacro)
@@ -39,4 +39,7 @@
       </collision>
     </link>
+    <gazebo reference="solid_wood_block_${handle}">
+      <material>Gazebo/Wood</material>
+    </gazebo>
   </xacro:macro>
 </robot>
