Commit message: rviz launch

File: urdf/map.urdf (robot description, URDF)
Before this commit: robot competition_map, 2 links, 1 joints
Links:
- link map_part1: geometry collision mesh filename=package://ICRA2023_Quadruped_Competition/meshes/part/map_pa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; visual mesh filename=package://ICRA2023_Quadruped_Competition/meshes/part/map_pa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

File: urdf/maps/map_part.urdf.xacro (robot description, xacro)
@@ -23,8 +23,8 @@
         <geometry>
           <mesh
-            filename="package://ICRA2023_Quadruped_Competition/meshes/part/map_part.dae"/>
+            filename="package://ICRA2023_Quadruped_Competition/meshes/part/map_part.stl"/>
         </geometry>
         <material name="">
-          <!-- <color rgba="1.0 0.41 0.41 1" />-->
+          <color rgba="1.0 0.41 0.41 1" />
         </material>
       </visual>
@@ -35,5 +35,5 @@
         <geometry>
           <mesh
-            filename="package://ICRA2023_Quadruped_Competition/meshes/map_part.dae"/>
+            filename="package://ICRA2023_Quadruped_Competition/meshes/part/map_part.stl"/>
         </geometry>
         <material name="">

Commit message: redo

File: urdf/map.urdf (robot description, URDF)
Before this commit: robot competition_map, 2 links, 1 joints
Links:
- removed link 1200x2400_OSB1
- added link map_part1, mass 1; collision mesh filename=package://ICRA2023_Quadruped_Competition/meshes/part/map_pa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; visual mesh filename=package://ICRA2023_Quadruped_Competition/meshes/part/map_pa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
Joints:
- removed joint 1200x2400_OSB1_joint
- added joint map_part1_joint: type fixed, parent world, child map_part1, origin xyz=0 0 0 rpy=0.0 0.0 0.0
