Commit message: modify: static map

File: urdf/map.urdf.xacro (robot description, xacro)
@@ -1398,3 +1398,6 @@
 	<xacro:Plastic_Storage_Crate parent="world" handle="1249" position="0.43000006675720215 -0.6000022888183594 0.31501901149749756" orientation="3.1415926535894076 2.586841583107698e-05 3.1415926237874725"/>
 	<xacro:Plastic_Storage_Crate parent="world" handle="1250" position="-0.26999950408935547 -0.0500032901763916 0.06500989198684692" orientation="3.1415926535894076 2.586841583107698e-05 3.1415926237874725"/>
+    <gazebo>
+	<static>true</static>
+	</gazebo>
 </robot>

File: urdf/obstacles/Akro_mils.urdf.xacro (robot description, xacro)
@@ -47,4 +47,5 @@
     <gazebo reference="Akro_mils_${handle}">
       <material>Gazebo/RedBright</material>
+      <static>true</static>
     </gazebo>
   </xacro:macro>

File: urdf/obstacles/New_600x400_2way_Wooden_Pallet.urdf.xacro (robot description, xacro)
@@ -224,4 +224,5 @@
     <gazebo reference="New_600x400_2way_Wooden_Pallet_${handle}">
       <material>Gazebo/Wood</material>
+      <static>true</static>
     </gazebo>
   </xacro:macro>

File: urdf/obstacles/New_EURO_EPAL_Pallet.urdf.xacro (robot description, xacro)
@@ -191,4 +191,5 @@
     <gazebo reference="New_EURO_EPAL_Pallet_${handle}">
       <material>Gazebo/Wood</material>
+      <static>true</static>
     </gazebo>
   </xacro:macro>

File: urdf/obstacles/Nisopa_Kerb_Ramp.urdf.xacro (robot description, xacro)
@@ -11,10 +11,10 @@
       name="Nisopa_Kerb_Ramp_${handle}">
       <inertial>
-        <origin xyz="0 0 0.5" rpy="0 0 0"/>
+        <origin xyz="0 0 0" rpy="0 0 0"/>
         <mass value="1"/>
         <inertia
-      ixx="1.0" ixy="0.0" ixz="0.0"
-      iyy="1.0" iyz="0.0"
-      izz="1.0"/>
+      ixx="0.01" ixy="0.0" ixz="0.0"
+      iyy="0.01" iyz="0.0"
+      izz="0.01"/>
       </inertial>
       <visual>
@@ -35,4 +35,5 @@
     <gazebo reference="Nisopa_Kerb_Ramp_${handle}">
       <material>Gazebo/DarkGrey</material>
+      <static>true</static>
     </gazebo>
   <!-- collision links -->

File: urdf/obstacles/Plastic_Curb_Ramp.urdf.xacro (robot description, xacro)
@@ -10,10 +10,10 @@
       name="Plastic_Curb_Ramp_${handle}">
       <inertial>
-        <origin xyz="0 0 0.5" rpy="0 0 0"/>
+        <origin xyz="0 0 0" rpy="0 0 0"/>
         <mass value="1"/>
         <inertia
-      ixx="1.0" ixy="0.0" ixz="0.0"
-      iyy="1.0" iyz="0.0"
-      izz="1.0"/>
+      ixx="0.01" ixy="0.0" ixz="0.0"
+      iyy="0.01" iyz="0.0"
+      izz="0.01"/>
       </inertial>
       <visual>
@@ -43,4 +43,5 @@
     <gazebo reference="Plastic_Curb_Ramp_${handle}">
       <material>Gazebo/Grey</material>
+      <static>true</static>
     </gazebo>
   </xacro:macro>

File: urdf/obstacles/Plastic_Storage_Crate.urdf.xacro (robot description, xacro)
@@ -10,10 +10,10 @@
       name="Plastic_Storage_Crate_${handle}">
       <inertial>
-        <origin xyz="0 0 0.5" rpy="0 0 0"/>
+        <origin xyz="0 0 0" rpy="0 0 0"/>
         <mass value="1"/>
         <inertia
-      ixx="1.0" ixy="0.0" ixz="0.0"
-      iyy="1.0" iyz="0.0"
-      izz="1.0"/>
+      ixx="+1.000e-03" ixy="+7.433e-15" ixz="+0.000e+00"
+      iyy="+1.000e-03" iyz="-7.105e-15"
+      izz="+1.000e-03"/>
       </inertial>
       <visual>
@@ -47,4 +47,5 @@
     <gazebo reference="Plastic_Storage_Crate_${handle}">
       <material>Gazebo/BlueGlow</material>
+      <static>true</static>
     </gazebo>
   </xacro:macro>

File: urdf/obstacles/Plywood_16mm_sheet.urdf.xacro (robot description, xacro)
@@ -41,4 +41,5 @@
     <gazebo reference="Plywood_16mm_sheet_${handle}">
       <material>Gazebo/Wood</material>
+      <static>true</static>
     </gazebo>
   </xacro:macro>

File: urdf/obstacles/Plywood_3mm_sheet.urdf.xacro (robot description, xacro)
@@ -41,4 +41,5 @@
     <gazebo reference="Plywood_3mm_sheet_${handle}">
       <material>Gazebo/Wood</material>
+      <static>true</static>
     </gazebo>
   </xacro:macro>

File: urdf/obstacles/Plywood_wall.urdf.xacro (robot description, xacro)
@@ -10,10 +10,10 @@
       name="Plywood_wall_${handle}">
       <inertial>
-        <origin xyz="0 0 0.5" rpy="0 0 0"/>
+        <origin xyz="0 0 0" rpy="0 0 0"/>
         <mass value="1"/>
         <inertia
-      ixx="1.0" ixy="0.0" ixz="0.0"
-      iyy="1.0" iyz="0.0"
-      izz="1.0"/>
+      ixx="+2.951e-02" ixy="-1.848e-09" ixz="-8.978e-11"
+      iyy="+6.051e-02" iyz="-1.758e-09"
+      izz="+3.102e-02"/>
       </inertial>
       <visual>
@@ -40,4 +40,5 @@
     <gazebo reference="Plywood_wall_${handle}">
       <material>Gazebo/Wood</material>
+      <static>true</static>
     </gazebo>
   </xacro:macro>

File: urdf/obstacles/seat_pad.urdf.xacro (robot description, xacro)
@@ -47,4 +47,5 @@
     <gazebo reference="Plastic_Storage_Crate_${handle}">
       <material>Gazebo/Grey</material>
+      <static>true</static>
     </gazebo>
   </xacro:macro>

File: urdf/obstacles/seat_pad_inner_compound.urdf.xacro (robot description, xacro)
@@ -43,4 +43,5 @@
     <gazebo reference="Plastic_Storage_Crate_${handle}">
       <material>Gazebo/Grey</material>
+      <static>true</static>
     </gazebo>
   </xacro:macro>

File: urdf/obstacles/seat_pad_outer_compound.urdf.xacro (robot description, xacro)
@@ -43,4 +43,5 @@
     <gazebo reference="Plastic_Storage_Crate_${handle}">
       <material>Gazebo/Grey</material>
+      <static>true</static>
     </gazebo>
   </xacro:macro>

File: urdf/obstacles/solid_wood_block.urdf.xacro (robot description, xacro)
@@ -10,10 +10,10 @@
       name="solid_wood_block_${handle}">
       <inertial>
-        <origin xyz="0 0 0.5" rpy="0 0 0"/>
+        <origin xyz="0 0 0" rpy="0 0 0"/>
         <mass value="1"/>
         <inertia
-      ixx="1.0" ixy="0.0" ixz="0.0"
-      iyy="1.0" iyz="0.0"
-      izz="1.0"/>
+      ixx="0.01" ixy="0.0" ixz="0.0"
+      iyy="0.01" iyz="0.0"
+      izz="0.01"/>
       </inertial>
       <visual>
@@ -41,4 +41,5 @@
     <gazebo reference="solid_wood_block_${handle}">
       <material>Gazebo/Wood</material>
+      <static>false</static>
     </gazebo>
   </xacro:macro>

File: urdf/test/map.urdf.xacro (robot description, xacro)
@@ -1,4 +1,7 @@
 <?xml version="1.0" ?>
 <robot xmlns:xacro="http://ros.org/wiki/xacro" name="competition_map_inner">
+	<gazebo>
+	<static>true</static>
+	</gazebo>
 	<link name="world"/>
 	<xacro:include filename="$(find ICRA2023_Quadruped_Competition)/urdf/obstacles/materials.xacro" />

File: urdf/test/terrain1_inner.urdf.xacro (robot description, xacro)
@@ -10,10 +10,10 @@
       name="terrain1_inner_${handle}">
       <inertial>
-        <origin xyz="0 0 0.5" rpy="0 0 0"/>
+        <origin xyz="0 0 0" rpy="0 0 0"/>
         <mass value="1"/>
         <inertia
-      ixx="1.0" ixy="0.0" ixz="0.0"
-      iyy="1.0" iyz="0.0"
-      izz="1.0"/>
+      ixx="0.01" ixy="0.0" ixz="0.0"
+      iyy="0.01" iyz="0.0"
+      izz="0.01"/>
       </inertial>
       <visual>
@@ -43,4 +43,5 @@
     <gazebo reference="terrain1_inner_${handle}">
       <material>Gazebo/Wood</material>
+      <static>true</static>
     </gazebo>
   </xacro:macro>

File: urdf/test/terrain2_inner.urdf.xacro (robot description, xacro)
@@ -10,10 +10,10 @@
       name="terrain2_inner_${handle}">
       <inertial>
-        <origin xyz="0 0 0.5" rpy="0 0 0"/>
+        <origin xyz="0 0 0" rpy="0 0 0"/>
         <mass value="1"/>
         <inertia
-      ixx="1.0" ixy="0.0" ixz="0.0"
-      iyy="1.0" iyz="0.0"
-      izz="1.0"/>
+      ixx="0.01" ixy="0.0" ixz="0.0"
+      iyy="0.01" iyz="0.0"
+      izz="0.01"/>
       </inertial>
       <visual>
@@ -43,4 +43,5 @@
     <gazebo reference="terrain2_inner_${handle}">
       <material>Gazebo/Wood</material>
+      <static>true</static>
     </gazebo>
   </xacro:macro>

File: urdf/test/terrain3_inner.urdf.xacro (robot description, xacro)
@@ -10,10 +10,10 @@
       name="terrain3_inner_${handle}">
       <inertial>
-        <origin xyz="0 0 0.5" rpy="0 0 0"/>
+        <origin xyz="0 0 0" rpy="0 0 0"/>
         <mass value="1"/>
         <inertia
-      ixx="1.0" ixy="0.0" ixz="0.0"
-      iyy="1.0" iyz="0.0"
-      izz="1.0"/>
+      ixx="0.01" ixy="0.0" ixz="0.0"
+      iyy="0.01" iyz="0.0"
+      izz="0.01"/>
       </inertial>
       <visual>
@@ -43,4 +43,5 @@
     <gazebo reference="terrain3_inner_${handle}">
       <material>Gazebo/Wood</material>
+      <static>true</static>
     </gazebo>
   </xacro:macro>

File: urdf/test/terrain3_inner2.urdf.xacro (robot description, xacro)
@@ -10,10 +10,10 @@
       name="terrain3_inner2_${handle}">
       <inertial>
-        <origin xyz="0 0 0.5" rpy="0 0 0"/>
+        <origin xyz="0 0 0" rpy="0 0 0"/>
         <mass value="1"/>
         <inertia
-      ixx="1.0" ixy="0.0" ixz="0.0"
-      iyy="1.0" iyz="0.0"
-      izz="1.0"/>
+      ixx="0.01" ixy="0.0" ixz="0.0"
+      iyy="0.01" iyz="0.0"
+      izz="0.01"/>
       </inertial>
       <visual>
@@ -43,4 +43,5 @@
     <gazebo reference="terrain3_inner2_${handle}">
       <material>Gazebo/DarkGrey</material>
+      <static>true</static>
     </gazebo>
   </xacro:macro>

File: urdf/test/terrain4_inner.urdf.xacro (robot description, xacro)
@@ -10,10 +10,10 @@
       name="terrain4_inner_${handle}">
       <inertial>
-        <origin xyz="0 0 0.5" rpy="0 0 0"/>
+        <origin xyz="0 0 0" rpy="0 0 0"/>
         <mass value="1"/>
         <inertia
-      ixx="1.0" ixy="0.0" ixz="0.0"
-      iyy="1.0" iyz="0.0"
-      izz="1.0"/>
+      ixx="0.01" ixy="0.0" ixz="0.0"
+      iyy="0.01" iyz="0.0"
+      izz="0.01"/>
       </inertial>
       <visual>
@@ -43,4 +43,5 @@
     <gazebo reference="terrain4_inner_${handle}">
       <material>Gazebo/Wood</material>
+      <static>true</static>
     </gazebo>
   </xacro:macro>
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
Commit message: add: gazebo world

File: urdf/map.urdf.xacro (robot description, xacro)
@@ -4,3 +4,6 @@
 	<xacro:include filename="$(find ICRA2023_Quadruped_Competition)/urdf/maps/map_part.urdf.xacro"/>
 	<xacro:map_part parent="world" handle="1" position="0 0 0" orientation="0.0 0.0 0.0"/>
+	<gazebo>
+		<static>true</static>
+	</gazebo>
 </robot>

File: urdf/maps/map_part.urdf.xacro (robot description, xacro)
@@ -43,4 +43,6 @@
     </link>
     <gazebo reference="map_part${handle}">
+      <material>Gazebo/Wood</material>
+      <static>true</static>
     </gazebo>
   </xacro:macro>
