Commit message: add: urdf.xacro

File: urdf/map.urdf.xacro (robot description, xacro)
@@ -2,6 +2,3875 @@
 <robot xmlns:xacro="http://ros.org/wiki/xacro" name="competition_map">
 	<link name="world"/>
-	<xacro:include filename="$(find ICRA2023_Quadruped_Competition)/urdf/obstacles/1200x2400_OSB.urdf.xacro"/>
-	<xacro:obj_1200x2400_OSB parent="world" handle="1" position="0 0 0" orientation="0.0 0.0 0.0"/>
+	<!-- 1200x2400_OSB__188889_ -->
+	<xacro:include filename="$(find ICRA2023_Quadruped_Competition)/urdf/obstacles/1200x2400_OSB__188889_.urdf.xacro"/>
+	<!-- 1200x2400_OSB__189837_ -->
+	<xacro:include filename="$(find ICRA2023_Quadruped_Competition)/urdf/obstacles/1200x2400_OSB__189837_.urdf.xacro"/>
+	<!-- 1200x2400_OSB__189840_ -->
+	<xacro:include filename="$(find ICRA2023_Quadruped_Competition)/urdf/obstacles/1200x2400_OSB__189840_.urdf.xacro"/>
+	<!-- 1200x2400_OSB__189843_ -->
+	<xacro:include filename="$(find ICRA2023_Quadruped_Competition)/urdf/obstacles/1200x2400_OSB__189843_.urdf.xacro"/>
+	<!-- 1200x2400_OSB__189846_ -->
+	<xacro:include filename="$(find ICRA2023_Quadruped_Competition)/urdf/obstacles/1200x2400_OSB__189846_.urdf.xacro"/>
+	<!-- 1200x2400_OSB__189909_ -->
+	<xacro:include filename="$(find ICRA2023_Quadruped_Competition)/urdf/obstacles/1200x2400_OSB__189909_.urdf.xacro"/>
+	<!-- 1200x2400_OSB__230819_ -->
+	<xacro:include filename="$(find ICRA2023_Quadruped_Competition)/urdf/obstacles/1200x2400_OSB__230819_.urdf.xacro"/>
+	<!-- 1200x2400_OSB__230837_ -->
+	<xacro:include filename="$(find ICRA2023_Quadruped_Competition)/urdf/obstacles/1200x2400_OSB__230837_.urdf.xacro"/>
+	<!-- 1200x600_OSB__194196_ -->
+	<xacro:include filename="$(find ICRA2023_Quadruped_Competition)/urdf/obstacles/1200x600_OSB__194196_.urdf.xacro"/>
+	<!-- 1200x600_OSB__194202_ -->
+	<xacro:include filename="$(find ICRA2023_Quadruped_Competition)/urdf/obstacles/1200x600_OSB__194202_.urdf.xacro"/>
+	<!-- 1200x600_OSB__230780_ -->
+	<xacro:include filename="$(find ICRA2023_Quadruped_Competition)/urdf/obstacles/1200x600_OSB__230780_.urdf.xacro"/>
+	<!-- 1200x600_OSB__230798_ -->
+	<xacro:include filename="$(find ICRA2023_Quadruped_Competition)/urdf/obstacles/1200x600_OSB__230798_.urdf.xacro"/>
+	<!-- 1200x600_OSB__231052_ -->
+	<xacro:include filename="$(find ICRA2023_Quadruped_Competition)/urdf/obstacles/1200x600_OSB__231052_.urdf.xacro"/>
+	<!-- 1200x600_OSB__231055_ -->
+	<xacro:include filename="$(find ICRA2023_Quadruped_Competition)/urdf/obstacles/1200x600_OSB__231055_.urdf.xacro"/>
+	<!-- 1200x600_OSB__231064_ -->
+	<xacro:include filename="$(find ICRA2023_Quadruped_Competition)/urdf/obstacles/1200x600_OSB__231064_.urdf.xacro"/>
+	<!-- 1200x600_OSB__231067_ -->
+	<xacro:include filename="$(find ICRA2023_Quadruped_Competition)/urdf/obstacles/1200x600_OSB__231067_.urdf.xacro"/>
+	<!-- 1200x600_OSB__231082_ -->
+	<xacro:include filename="$(find ICRA2023_Quadruped_Competition)/urdf/obstacles/1200x600_OSB__231082_.urdf.xacro"/>
+	<!-- 1200x600_OSB__231097_ -->
+	<xacro:include filename="$(find ICRA2023_Quadruped_Competition)/urdf/obstacles/1200x600_OSB__231097_.urdf.xacro"/>
+	<!-- 1200x600_OSB__231100_ -->
+	<xacro:include filename="$(find ICRA2023_Quadruped_Competition)/urdf/obstacles/1200x600_OSB__231100_.urdf.xacro"/>
+	<!-- 1200x600_OSB__231112_ -->
+	<xacro:include filename="$(find ICRA2023_Quadruped_Competition)/urdf/obstacles/1200x600_OSB__231112_.urdf.xacro"/>
+	<!-- 1200x600_OSB__231121_ -->
+	<xacro:include filename="$(find ICRA2023_Quadruped_Competition)/urdf/obstacles/1200x600_OSB__231121_.urdf.xacro"/>
+	<!-- 1200x600_OSB__231127_ -->
+	<xacro:include filename="$(find ICRA2023_Quadruped_Competition)/urdf/obstacles/1200x600_OSB__231127_.urdf.xacro"/>
+	<!-- 1200x600_OSB__231136_ -->
+	<xacro:include filename="$(find ICRA2023_Quadruped_Competition)/urdf/obstacles/1200x600_OSB__231136_.urdf.xacro"/>
+	<!-- 1200x600_OSB__231139_ -->
+	<xacro:include filename="$(find ICRA2023_Quadruped_Competition)/urdf/obstacles/1200x600_OSB__231139_.urdf.xacro"/>
+	<!-- 1200x600_OSB__231148_ -->
+	<xacro:include filename="$(find ICRA2023_Quadruped_Competition)/urdf/obstacles/1200x600_OSB__231148_.urdf.xacro"/>
+	<!-- 1200x600_OSB__231151_ -->
+	<xacro:include filename="$(find ICRA2023_Quadruped_Competition)/urdf/obstacles/1200x600_OSB__231151_.urdf.xacro"/>
+	<!-- 12_00x1200_OSB_1__192425_ -->
+	<xacro:include filename="$(find ICRA2023_Quadruped_Competition)/urdf/obstacles/12_00x1200_OSB_1__192425_.urdf.xacro"/>
+	<!-- 12_00x1200_OSB__162540_ -->
+	<xacro:include filename="$(find ICRA2023_Quadruped_Competition)/urdf/obstacles/12_00x1200_OSB__162540_.urdf.xacro"/>
+	<!-- 12_00x1200_OSB__192655_ -->
+	<xacro:include filename="$(find ICRA2023_Quadruped_Competition)/urdf/obstacles/12_00x1200_OSB__192655_.urdf.xacro"/>
+	<!-- 12_00x1200_OSB__192674_ -->
+	<xacro:include filename="$(find ICRA2023_Quadruped_Competition)/urdf/obstacles/12_00x1200_OSB__192674_.urdf.xacro"/>
+	<!-- 12_00x1200_OSB__194011_ -->
+	<xacro:include filename="$(find ICRA2023_Quadruped_Competition)/urdf/obstacles/12_00x1200_OSB__194011_.urdf.xacro"/>
+	<!-- 12_00x1200_OSB__194014_ -->
+	<xacro:include filename="$(find ICRA2023_Quadruped_Competition)/urdf/obstacles/12_00x1200_OSB__194014_.urdf.xacro"/>
+	<!-- 12_00x1200_OSB__231103_ -->
+	<xacro:include filename="$(find ICRA2023_Quadruped_Competition)/urdf/obstacles/12_00x1200_OSB__231103_.urdf.xacro"/>
+	<!-- 12_00x1200_OSB__231118_ -->
+	<xacro:include filename="$(find ICRA2023_Quadruped_Competition)/urdf/obstacles/12_00x1200_OSB__231118_.urdf.xacro"/>
+	<!-- 1_1m_5x10cm_beam__188883_ -->
+	<xacro:include filename="$(find ICRA2023_Quadruped_Competition)/urdf/obstacles/1_1m_5x10cm_beam__188883_.urdf.xacro"/>
+	<!-- 1_1m_5x10cm_beam__188904_ -->
+	<xacro:include filename="$(find ICRA2023_Quadruped_Competition)/urdf/obstacles/1_1m_5x10cm_beam__188904_.urdf.xacro"/>
+	<!-- 1_1m_5x10cm_beam__189849_ -->
+	<xacro:include filename="$(find ICRA2023_Quadruped_Competition)/urdf/obstacles/1_1m_5x10cm_beam__189849_.urdf.xacro"/>
+	<!-- 1_1m_5x10cm_beam__189852_ -->
+	<xacro:include filename="$(find ICRA2023_Quadruped_Competition)/urdf/obstacles/1_1m_5x10cm_beam__189852_.urdf.xacro"/>
+	<!-- 1_1m_5x10cm_beam__189855_ -->
+	<xacro:include filename="$(find ICRA2023_Quadruped_Competition)/urdf/obstacles/1_1m_5x10cm_beam__189855_.urdf.xacro"/>
+	<!-- 1_1m_5x10cm_beam__189858_ -->
+	<xacro:include filename="$(find ICRA2023_Quadruped_Competition)/urdf/obstacles/1_1m_5x10cm_beam__189858_.urdf.xacro"/>
+	<!-- 1_1m_5x10cm_beam__189861_ -->
+	<xacro:include filename="$(find ICRA2023_Quadruped_Competition)/urdf/obstacles/1_1m_5x10cm_beam__189861_.urdf.xacro"/>
+	<!-- 1_1m_5x10cm_beam__189864_ -->
+	<xacro:include filename="$(find ICRA2023_Quadruped_Competition)/urdf/obstacles/1_1m_5x10cm_beam__189864_.urdf.xacro"/>
+	<!-- 1_1m_5x10cm_beam__189867_ -->
+	<xacro:include filename="$(find ICRA2023_Quadruped_Competition)/urdf/obstacles/1_1m_5x10cm_beam__189867_.urdf.xacro"/>
+	<!-- 1_1m_5x10cm_beam__189870_ -->
+	<xacro:include filename="$(find ICRA2023_Quadruped_Competition)/urdf/obstacles/1_1m_5x10cm_beam__189870_.urdf.xacro"/>
+	<!-- 1_1m_5x10cm_beam__225755_ -->
+	<xacro:include filename="$(find ICRA2023_Quadruped_Competition)/urdf/obstacles/1_1m_5x10cm_beam__225755_.urdf.xacro"/>
+	<!-- 1_1m_5x10cm_beam__225758_ -->
+	<xacro:include filename="$(find ICRA2023_Quadruped_Competition)/urdf/obstacles/1_1m_5x10cm_beam__225758_.urdf.xacro"/>
+	<!-- 1_1m_5x10cm_beam__225761_ -->
+	<xacro:include filename="$(find ICRA2023_Quadruped_Competition)/urdf/obstacles/1_1m_5x10cm_beam__225761_.urdf.xacro"/>
+	<!-- 1_1m_5x10cm_beam__225785_ -->
+	<xacro:include filename="$(find ICRA2023_Quadruped_Competition)/urdf/obstacles/1_1m_5x10cm_beam__225785_.urdf.xacro"/>
+	<!-- 1_1m_5x10cm_beam__225788_ -->
+	<xacro:include filename="$(find ICRA2023_Quadruped_Competition)/urdf/obstacles/1_1m_5x10cm_beam__225788_.urdf.xacro"/>
+	<!-- 1_1m_5x10cm_beam__230822_ -->
+	<xacro:include filename="$(find ICRA2023_Quadruped_Competition)/urdf/obstacles/1_1m_5x10cm_beam__230822_.urdf.xacro"/>
+	<!-- 1_1m_5x10cm_beam__230828_ -->
+	<xacro:include filename="$(find ICRA2023_Quadruped_Competition)/urdf/obstacles/1_1m_5x10cm_beam__230828_.urdf.xacro"/>
+	<!-- 1_1m_5x10cm_beam__230834_ -->
+	<xacro:include filename="$(find ICRA2023_Quadruped_Competition)/urdf/obstacles/1_1m_5x10cm_beam__230834_.urdf.xacro"/>
+	<!-- 1_1m_5x10cm_beam__230855_ -->
+	<xacro:include filename="$(find ICRA2023_Quadruped_Competition)/urdf/obstacles/1_1m_5x10cm_beam__230855_.urdf.xacro"/>
+	<!-- 1_2m_5x10cm_beam_1__225776_ -->
+	<xacro:include filename="$(find ICRA2023_Quadruped_Competition)/urdf/obstacles/1_2m_5x10cm_beam_1__225776_.urdf.xacro"/>
+	<!-- 1_2m_5x10cm_beam_1__225794_ -->
+	<xacro:include filename="$(find ICRA2023_Quadruped_Competition)/urdf/obstacles/1_2m_5x10cm_beam_1__225794_.urdf.xacro"/>
+	<!-- 1_2m_5x10cm_beam_1__231049_ -->
+	<xacro:include filename="$(find ICRA2023_Quadruped_Competition)/urdf/obstacles/1_2m_5x10cm_beam_1__231049_.urdf.xacro"/>
+	<!-- 1_2m_5x10cm_beam_1__231073_ -->
+	<xacro:include filename="$(find ICRA2023_Quadruped_Competition)/urdf/obstacles/1_2m_5x10cm_beam_1__231073_.urdf.xacro"/>
+	<!-- 1_2m_5x10cm_beam_1__231076_ -->
+	<xacro:include filename="$(find ICRA2023_Quadruped_Competition)/urdf/obstacles/1_2m_5x10cm_beam_1__231076_.urdf.xacro"/>
+	<!-- 1_2m_5x10cm_beam_1__231079_ -->
+	<xacro:include filename="$(find ICRA2023_Quadruped_Competition)/urdf/obstacles/1_2m_5x10cm_beam_1__231079_.urdf.xacro"/>
+	<!-- 1_2m_5x10cm_beam__225749_ -->
+	<xacro:include filename="$(find ICRA2023_Quadruped_Competition)/urdf/obstacles/1_2m_5x10cm_beam__225749_.urdf.xacro"/>
+	<!-- 1_2m_5x10cm_beam__225752_ -->
+	<xacro:include filename="$(find ICRA2023_Quadruped_Competition)/urdf/obstacles/1_2m_5x10cm_beam__225752_.urdf.xacro"/>
+	<!-- 1__188078_ -->
+	<xacro:include filename="$(find ICRA2023_Quadruped_Competition)/urdf/obstacles/1__188078_.urdf.xacro"/>
+	<!-- 1__188081_ -->
+	<xacro:include filename="$(find ICRA2023_Quadruped_Competition)/urdf/obstacles/1__188081_.urdf.xacro"/>
+	<!-- 2_4m_5x10cm_beam__188898_ -->
+	<xacro:include filename="$(find ICRA2023_Quadruped_Competition)/urdf/obstacles/2_4m_5x10cm_beam__188898_.urdf.xacro"/>
+	<!-- 2_4m_5x10cm_beam__188901_ -->
+	<xacro:include filename="$(find ICRA2023_Quadruped_Competition)/urdf/obstacles/2_4m_5x10cm_beam__188901_.urdf.xacro"/>
+	<!-- 2_4m_5x10cm_beam__189873_ -->
+	<xacro:include filename="$(find ICRA2023_Quadruped_Competition)/urdf/obstacles/2_4m_5x10cm_beam__189873_.urdf.xacro"/>
+	<!-- 2_4m_5x10cm_beam__189876_ -->
+	<xacro:include filename="$(find ICRA2023_Quadruped_Competition)/urdf/obstacles/2_4m_5x10cm_beam__189876_.urdf.xacro"/>
+	<!-- 2_4m_5x10cm_beam__189879_ -->
+	<xacro:include filename="$(find ICRA2023_Quadruped_Competition)/urdf/obstacles/2_4m_5x10cm_beam__189879_.urdf.xacro"/>
+	<!-- 2_4m_5x10cm_beam__189882_ -->
+	<xacro:include filename="$(find ICRA2023_Quadruped_Competition)/urdf/obstacles/2_4m_5x10cm_beam__189882_.urdf.xacro"/>
+	<!-- 2_4m_5x10cm_beam__189885_ -->
+	<xacro:include filename="$(find ICRA2023_Quadruped_Competition)/urdf/obstacles/2_4m_5x10cm_beam__189885_.urdf.xacro"/>
+	<!-- 2_4m_5x10cm_beam__189888_ -->
+	<xacro:include filename="$(find ICRA2023_Quadruped_Competition)/urdf/obstacles/2_4m_5x10cm_beam__189888_.urdf.xacro"/>
+	<!-- 2_4m_5x10cm_beam__189891_ -->
+	<xacro:include filename="$(find ICRA2023_Quadruped_Competition)/urdf/obstacles/2_4m_5x10cm_beam__189891_.urdf.xacro"/>
+	<!-- 2_4m_5x10cm_beam__189894_ -->
+	<xacro:include filename="$(find ICRA2023_Quadruped_Competition)/urdf/obstacles/2_4m_5x10cm_beam__189894_.urdf.xacro"/>
+	<!-- 2_4m_5x10cm_beam__230831_ -->
+	<xacro:include filename="$(find ICRA2023_Quadruped_Competition)/urdf/obstacles/2_4m_5x10cm_beam__230831_.urdf.xacro"/>
+	<!-- 2_4m_5x10cm_beam__230843_ -->
+	<xacro:include filename="$(find ICRA2023_Quadruped_Competition)/urdf/obstacles/2_4m_5x10cm_beam__230843_.urdf.xacro"/>
+	<!-- 2_4m_5x10cm_beam__230846_ -->
+	<xacro:include filename="$(find ICRA2023_Quadruped_Competition)/urdf/obstacles/2_4m_5x10cm_beam__230846_.urdf.xacro"/>
+	<!-- 2_4m_5x10cm_beam__230849_ -->
+	<xacro:include filename="$(find ICRA2023_Quadruped_Competition)/urdf/obstacles/2_4m_5x10cm_beam__230849_.urdf.xacro"/>
+	<!-- 2__188018_ -->
+	<xacro:include filename="$(find ICRA2023_Quadruped_Competition)/urdf/obstacles/2__188018_.urdf.xacro"/>
+	<!-- 2__188021_ -->
+	<xacro:include filename="$(find ICRA2023_Quadruped_Competition)/urdf/obstacles/2__188021_.urdf.xacro"/>
+	<!-- 300x600_OSB__188907_ -->
+	<xacro:include filename="$(find ICRA2023_Quadruped_Competition)/urdf/obstacles/300x600_OSB__188907_.urdf.xacro"/>
+	<!-- 300x600_OSB__194199_ -->
+	<xacro:include filename="$(find ICRA2023_Quadruped_Competition)/urdf/obstacles/300x600_OSB__194199_.urdf.xacro"/>
+	<!-- 300x600_OSB__194205_ -->
+	<xacro:include filename="$(find ICRA2023_Quadruped_Competition)/urdf/obstacles/300x600_OSB__194205_.urdf.xacro"/>
+	<!-- 300x600_OSB__194208_ -->
+	<xacro:include filename="$(find ICRA2023_Quadruped_Competition)/urdf/obstacles/300x600_OSB__194208_.urdf.xacro"/>
+	<!-- 300x600_OSB__194217_ -->
+	<xacro:include filename="$(find ICRA2023_Quadruped_Competition)/urdf/obstacles/300x600_OSB__194217_.urdf.xacro"/>
+	<!-- 300x600_OSB__230801_ -->
+	<xacro:include filename="$(find ICRA2023_Quadruped_Competition)/urdf/obstacles/300x600_OSB__230801_.urdf.xacro"/>
+	<!-- 300x600_OSB__230810_ -->
+	<xacro:include filename="$(find ICRA2023_Quadruped_Competition)/urdf/obstacles/300x600_OSB__230810_.urdf.xacro"/>
+	<!-- 3__187996_ -->
+	<xacro:include filename="$(find ICRA2023_Quadruped_Competition)/urdf/obstacles/3__187996_.urdf.xacro"/>
+	<!-- 3__187999_ -->
+	<xacro:include filename="$(find ICRA2023_Quadruped_Competition)/urdf/obstacles/3__187999_.urdf.xacro"/>
+	<!-- 42'_2x2_baluster__188128_ -->
+	<xacro:include filename="$(find ICRA2023_Quadruped_Competition)/urdf/obstacles/42'_2x2_baluster__188128_.urdf.xacro"/>
+	<!-- 450mm_hurdle_retainer__231166_ -->
+	<xacro:include filename="$(find ICRA2023_Quadruped_Competition)/urdf/obstacles/450mm_hurdle_retainer__231166_.urdf.xacro"/>
+	<!-- 450mm_hurdle_retainer__231169_ -->
+	<xacro:include filename="$(find ICRA2023_Quadruped_Competition)/urdf/obstacles/450mm_hurdle_retainer__231169_.urdf.xacro"/>
+	<!-- 450mm_hurdle_retainer__231172_ -->
+	<xacro:include filename="$(find ICRA2023_Quadruped_Competition)/urdf/obstacles/450mm_hurdle_retainer__231172_.urdf.xacro"/>
+	<!-- 450mm_hurdle_retainer__231175_ -->
+	<xacro:include filename="$(find ICRA2023_Quadruped_Competition)/urdf/obstacles/450mm_hurdle_retainer__231175_.urdf.xacro"/>
+	<!-- 450mm_hurdle_retainer__231178_ -->
+	<xacro:include filename="$(find ICRA2023_Quadruped_Competition)/urdf/obstacles/450mm_hurdle_retainer__231178_.urdf.xacro"/>
+	<!-- 450mm_hurdle_retainer__231181_ -->
+	<xacro:include filename="$(find ICRA2023_Quadruped_Competition)/urdf/obstacles/450mm_hurdle_retainer__231181_.urdf.xacro"/>
+	<!-- 450mm_hurdle_retainer__231184_ -->
+	<xacro:include filename="$(find ICRA2023_Quadruped_Competition)/urdf/obstacles/450mm_hurdle_retainer__231184_.urdf.xacro"/>
+	<!-- 450mm_hurdle_retainer__231187_ -->
+	<xacro:include filename="$(find ICRA2023_Quadruped_Competition)/urdf/obstacles/450mm_hurdle_retainer__231187_.urdf.xacro"/>
+	<!-- 450mm_hurdle_retainer__231190_ -->
+	<xacro:include filename="$(find ICRA2023_Quadruped_Competition)/urdf/obstacles/450mm_hurdle_retainer__231190_.urdf.xacro"/>
+	<!-- 450mm_hurdle_retainer__231193_ -->
+	<xacro:include filename="$(find ICRA2023_Quadruped_Competition)/urdf/obstacles/450mm_hurdle_retainer__231193_.urdf.xacro"/>
+	<!-- 450mm_hurdle_retainer__231196_ -->
+	<xacro:include filename="$(find ICRA2023_Quadruped_Competition)/urdf/obstacles/450mm_hurdle_retainer__231196_.urdf.xacro"/>
+	<!-- 450mm_hurdle_retainer__231199_ -->
+	<xacro:include filename="$(find ICRA2023_Quadruped_Competition)/urdf/obstacles/450mm_hurdle_retainer__231199_.urdf.xacro"/>
+	<!-- 450mm_hurdle_retainer__231202_ -->
+	<xacro:include filename="$(find ICRA2023_Quadruped_Competition)/urdf/obstacles/450mm_hurdle_retainer__231202_.urdf.xacro"/>
+	<!-- 450mm_hurdle_retainer__231205_ -->
+	<xacro:include filename="$(find ICRA2023_Quadruped_Competition)/urdf/obstacles/450mm_hurdle_retainer__231205_.urdf.xacro"/>
+	<!-- 4_1__188056_ -->
+	<xacro:include filename="$(find ICRA2023_Quadruped_Competition)/urdf/obstacles/4_1__188056_.urdf.xacro"/>
+	<!-- 4_1__188059_ -->
+	<xacro:include filename="$(find ICRA2023_Quadruped_Competition)/urdf/obstacles/4_1__188059_.urdf.xacro"/>
+	<!-- 5x5x30_cm_wall_corner__188886_ -->
+	<xacro:include filename="$(find ICRA2023_Quadruped_Competition)/urdf/obstacles/5x5x30_cm_wall_corner__188886_.urdf.xacro"/>
+	<!-- 5x5x30_cm_wall_corner__188910_ -->
+	<xacro:include filename="$(find ICRA2023_Quadruped_Competition)/urdf/obstacles/5x5x30_cm_wall_corner__188910_.urdf.xacro"/>
+	<!-- 5x5x30_cm_wall_corner__194172_ -->
+	<xacro:include filename="$(find ICRA2023_Quadruped_Competition)/urdf/obstacles/5x5x30_cm_wall_corner__194172_.urdf.xacro"/>
+	<!-- 5x5x30_cm_wall_corner__194175_ -->
+	<xacro:include filename="$(find ICRA2023_Quadruped_Competition)/urdf/obstacles/5x5x30_cm_wall_corner__194175_.urdf.xacro"/>
+	<!-- 5x5x30_cm_wall_corner__194178_ -->
+	<xacro:include filename="$(find ICRA2023_Quadruped_Competition)/urdf/obstacles/5x5x30_cm_wall_corner__194178_.urdf.xacro"/>
+	<!-- 5x5x30_cm_wall_corner__194181_ -->
+	<xacro:include filename="$(find ICRA2023_Quadruped_Competition)/urdf/obstacles/5x5x30_cm_wall_corner__194181_.urdf.xacro"/>
+	<!-- 5x5x30_cm_wall_corner__194184_ -->
+	<xacro:include filename="$(find ICRA2023_Quadruped_Competition)/urdf/obstacles/5x5x30_cm_wall_corner__194184_.urdf.xacro"/>
+	<!-- 5x5x30_cm_wall_corner__194187_ -->
+	<xacro:include filename="$(find ICRA2023_Quadruped_Competition)/urdf/obstacles/5x5x30_cm_wall_corner__194187_.urdf.xacro"/>
+	<!-- 5x5x30_cm_wall_corner__194190_ -->
+	<xacro:include filename="$(find ICRA2023_Quadruped_Competition)/urdf/obstacles/5x5x30_cm_wall_corner__194190_.urdf.xacro"/>
+	<!-- 5x5x30_cm_wall_corner__194193_ -->
+	<xacro:include filename="$(find ICRA2023_Quadruped_Competition)/urdf/obstacles/5x5x30_cm_wall_corner__194193_.urdf.xacro"/>
+	<!-- 5x5x30_cm_wall_corner__194211_ -->
+	<xacro:include filename="$(find ICRA2023_Quadruped_Competition)/urdf/obstacles/5x5x30_cm_wall_corner__194211_.urdf.xacro"/>
+	<!-- 5x5x30_cm_wall_corner__194214_ -->
+	<xacro:include filename="$(find ICRA2023_Quadruped_Competition)/urdf/obstacles/5x5x30_cm_wall_corner__194214_.urdf.xacro"/>
+	<!-- 5x5x30_cm_wall_corner__230777_ -->
+	<xacro:include filename="$(find ICRA2023_Quadruped_Competition)/urdf/obstacles/5x5x30_cm_wall_corner__230777_.urdf.xacro"/>
+	<!-- 5x5x30_cm_wall_corner__230783_ -->
+	<xacro:include filename="$(find ICRA2023_Quadruped_Competition)/urdf/obstacles/5x5x30_cm_wall_corner__230783_.urdf.xacro"/>
+	<!-- 5x5x30_cm_wall_corner__230786_ -->
+	<xacro:include filename="$(find ICRA2023_Quadruped_Competition)/urdf/obstacles/5x5x30_cm_wall_corner__230786_.urdf.xacro"/>
+	<!-- 5x5x30_cm_wall_corner__230807_ -->
+	<xacro:include filename="$(find ICRA2023_Quadruped_Competition)/urdf/obstacles/5x5x30_cm_wall_corner__230807_.urdf.xacro"/>
+	<!-- 600x1200_OSB__188892_ -->
+	<xacro:include filename="$(find ICRA2023_Quadruped_Competition)/urdf/obstacles/600x1200_OSB__188892_.urdf.xacro"/>
+	<!-- 600x1200_OSB__194139_ -->
+	<xacro:include filename="$(find ICRA2023_Quadruped_Competition)/urdf/obstacles/600x1200_OSB__194139_.urdf.xacro"/>
+	<!-- 600x1200_OSB__194142_ -->
+	<xacro:include filename="$(find ICRA2023_Quadruped_Competition)/urdf/obstacles/600x1200_OSB__194142_.urdf.xacro"/>
+	<!-- 600x1200_OSB__194154_ -->
+	<xacro:include filename="$(find ICRA2023_Quadruped_Competition)/urdf/obstacles/600x1200_OSB__194154_.urdf.xacro"/>
+	<!-- 600x1200_OSB__194157_ -->
+	<xacro:include filename="$(find ICRA2023_Quadruped_Competition)/urdf/obstacles/600x1200_OSB__194157_.urdf.xacro"/>
+	<!-- 600x1200_OSB__230789_ -->
+	<xacro:include filename="$(find ICRA2023_Quadruped_Competition)/urdf/obstacles/600x1200_OSB__230789_.urdf.xacro"/>
+	<!-- 600x1200_OSB__230795_ -->
+	<xacro:include filename="$(find ICRA2023_Quadruped_Competition)/urdf/obstacles/600x1200_OSB__230795_.urdf.xacro"/>
+	<!-- 600x2400_OSB__188895_ -->
+	<xacro:include filename="$(find ICRA2023_Quadruped_Competition)/urdf/obstacles/600x2400_OSB__188895_.urdf.xacro"/>
+	<!-- 600x2400_OSB__193609_ -->
+	<xacro:include filename="$(find ICRA2023_Quadruped_Competition)/urdf/obstacles/600x2400_OSB__193609_.urdf.xacro"/>
+	<!-- 600x2400_OSB__194133_ -->
+	<xacro:include filename="$(find ICRA2023_Quadruped_Competition)/urdf/obstacles/600x2400_OSB__194133_.urdf.xacro"/>
+	<!-- 600x2400_OSB__194145_ -->
+	<xacro:include filename="$(find ICRA2023_Quadruped_Competition)/urdf/obstacles/600x2400_OSB__194145_.urdf.xacro"/>
+	<!-- 600x2400_OSB__194148_ -->
+	<xacro:include filename="$(find ICRA2023_Quadruped_Competition)/urdf/obstacles/600x2400_OSB__194148_.urdf.xacro"/>
+	<!-- 600x2400_OSB__194151_ -->
+	<xacro:include filename="$(find ICRA2023_Quadruped_Competition)/urdf/obstacles/600x2400_OSB__194151_.urdf.xacro"/>
+	<!-- 600x2400_OSB__230792_ -->
+	<xacro:include filename="$(find ICRA2023_Quadruped_Competition)/urdf/obstacles/600x2400_OSB__230792_.urdf.xacro"/>
+	<!-- 600x2400_OSB__230804_ -->
+	<xacro:include filename="$(find ICRA2023_Quadruped_Competition)/urdf/obstacles/600x2400_OSB__230804_.urdf.xacro"/>
+	<!-- 600x2400_OSB__231085_ -->
+	<xacro:include filename="$(find ICRA2023_Quadruped_Competition)/urdf/obstacles/600x2400_OSB__231085_.urdf.xacro"/>
+	<!-- 600x2400_OSB__231088_ -->
+	<xacro:include filename="$(find ICRA2023_Quadruped_Competition)/urdf/obstacles/600x2400_OSB__231088_.urdf.xacro"/>
+	<!-- __127472_ -->
+	<xacro:include filename="$(find ICRA2023_Quadruped_Competition)/urdf/obstacles/__127472_.urdf.xacro"/>
+	<!-- __127478_ -->
+	<xacro:include filename="$(find ICRA2023_Quadruped_Competition)/urdf/obstacles/__127478_.urdf.xacro"/>
+	<!-- __127538_ -->
+	<xacro:include filename="$(find ICRA2023_Quadruped_Competition)/urdf/obstacles/__127538_.urdf.xacro"/>
+	<!-- __146947_ -->
+	<xacro:include filename="$(find ICRA2023_Quadruped_Competition)/urdf/obstacles/__146947_.urdf.xacro"/>
+	<!-- __187834_ -->
+	<xacro:include filename="$(find ICRA2023_Quadruped_Competition)/urdf/obstacles/__187834_.urdf.xacro"/>
+	<!-- Component_246__131227_ -->
+	<xacro:include filename="$(find ICRA2023_Quadruped_Competition)/urdf/obstacles/Component_246__131227_.urdf.xacro"/>
+	<!-- Component_246__131230_ -->
+	<xacro:include filename="$(find ICRA2023_Quadruped_Competition)/urdf/obstacles/Component_246__131230_.urdf.xacro"/>
+	<!-- Component_246__131233_ -->
+	<xacro:include filename="$(find ICRA2023_Quadruped_Competition)/urdf/obstacles/Component_246__131233_.urdf.xacro"/>
+	<!-- Component_246__131236_ -->
+	<xacro:include filename="$(find ICRA2023_Quadruped_Competition)/urdf/obstacles/Component_246__131236_.urdf.xacro"/>
+	<!-- Component_247__131299_ -->
+	<xacro:include filename="$(find ICRA2023_Quadruped_Competition)/urdf/obstacles/Component_247__131299_.urdf.xacro"/>
+	<!-- Component_247__131302_ -->
+	<xacro:include filename="$(find ICRA2023_Quadruped_Competition)/urdf/obstacles/Component_247__131302_.urdf.xacro"/>
+	<!-- Component_247__131305_ -->
+	<xacro:include filename="$(find ICRA2023_Quadruped_Competition)/urdf/obstacles/Component_247__131305_.urdf.xacro"/>
+	<!-- Component_247__131308_ -->
+	<xacro:include filename="$(find ICRA2023_Quadruped_Competition)/urdf/obstacles/Component_247__131308_.urdf.xacro"/>
+	<!-- Component_248__131251_ -->
+	<xacro:include filename="$(find ICRA2023_Quadruped_Competition)/urdf/obstacles/Component_248__131251_.urdf.xacro"/>
+	<!-- Component_248__131254_ -->
+	<xacro:include filename="$(find ICRA2023_Quadruped_Competition)/urdf/obstacles/Component_248__131254_.urdf.xacro"/>
+	<!-- Component_248__131257_ -->
+	<xacro:include filename="$(find ICRA2023_Quadruped_Competition)/urdf/obstacles/Component_248__131257_.urdf.xacro"/>
+	<!-- Component_248__131260_ -->
+	<xacro:include filename="$(find ICRA2023_Quadruped_Competition)/urdf/obstacles/Component_248__131260_.urdf.xacro"/>
+	<!-- Component_249__131275_ -->
+	<xacro:include filename="$(find ICRA2023_Quadruped_Competition)/urdf/obstacles/Component_249__131275_.urdf.xacro"/>
+	<!-- Component_249__131278_ -->
+	<xacro:include filename="$(find ICRA2023_Quadruped_Competition)/urdf/obstacles/Component_249__131278_.urdf.xacro"/>
+	<!-- Component_249__131281_ -->
+	<xacro:include filename="$(find ICRA2023_Quadruped_Competition)/urdf/obstacles/Component_249__131281_.urdf.xacro"/>
+	<!-- Component_249__131284_ -->
+	<xacro:include filename="$(find ICRA2023_Quadruped_Competition)/urdf/obstacles/Component_249__131284_.urdf.xacro"/>
+	<!-- Component_251__131209_ -->
+	<xacro:include filename="$(find ICRA2023_Quadruped_Competition)/urdf/obstacles/Component_251__131209_.urdf.xacro"/>
+	<!-- Component_251__131212_ -->
+	<xacro:include filename="$(find ICRA2023_Quadruped_Competition)/urdf/obstacles/Component_251__131212_.urdf.xacro"/>
+	<!-- Component_272__118757_ -->
+	<xacro:include filename="$(find ICRA2023_Quadruped_Competition)/urdf/obstacles/Component_272__118757_.urdf.xacro"/>
+	<!-- Component_272__118760_ -->
+	<xacro:include filename="$(find ICRA2023_Quadruped_Competition)/urdf/obstacles/Component_272__118760_.urdf.xacro"/>
+	<!-- Component_272__118763_ -->
+	<xacro:include filename="$(find ICRA2023_Quadruped_Competition)/urdf/obstacles/Component_272__118763_.urdf.xacro"/>
+	<!-- Component_272__118766_ -->
+	<xacro:include filename="$(find ICRA2023_Quadruped_Competition)/urdf/obstacles/Component_272__118766_.urdf.xacro"/>
+	<!-- Component_272__118769_ -->
+	<xacro:include filename="$(find ICRA2023_Quadruped_Competition)/urdf/obstacles/Component_272__118769_.urdf.xacro"/>
+	<!-- Component_272__118772_ -->
+	<xacro:include filename="$(find ICRA2023_Quadruped_Competition)/urdf/obstacles/Component_272__118772_.urdf.xacro"/>
+	<!-- Component_272__118775_ -->
+	<xacro:include filename="$(find ICRA2023_Quadruped_Competition)/urdf/obstacles/Component_272__118775_.urdf.xacro"/>
+	<!-- Component_2__225782_ -->
+	<xacro:include filename="$(find ICRA2023_Quadruped_Competition)/urdf/obstacles/Component_2__225782_.urdf.xacro"/>
+	<!-- Component_2__225791_ -->
+	<xacro:include filename="$(find ICRA2023_Quadruped_Competition)/urdf/obstacles/Component_2__225791_.urdf.xacro"/>
+	<!-- Component_363__187680_ -->
+	<xacro:include filename="$(find ICRA2023_Quadruped_Competition)/urdf/obstacles/Component_363__187680_.urdf.xacro"/>
+	<!-- Component_363__187683_ -->
+	<xacro:include filename="$(find ICRA2023_Quadruped_Competition)/urdf/obstacles/Component_363__187683_.urdf.xacro"/>
+	<!-- Component_7__189930_ -->
+	<xacro:include filename="$(find ICRA2023_Quadruped_Competition)/urdf/obstacles/Component_7__189930_.urdf.xacro"/>
+	<!-- Component_7__189933_ -->
+	<xacro:include filename="$(find ICRA2023_Quadruped_Competition)/urdf/obstacles/Component_7__189933_.urdf.xacro"/>
+	<!-- Component_7__189936_ -->
+	<xacro:include filename="$(find ICRA2023_Quadruped_Competition)/urdf/obstacles/Component_7__189936_.urdf.xacro"/>
+	<!-- Component_7__189939_ -->
+	<xacro:include filename="$(find ICRA2023_Quadruped_Competition)/urdf/obstacles/Component_7__189939_.urdf.xacro"/>
+	<!-- Component_7__189942_ -->
+	<xacro:include filename="$(find ICRA2023_Quadruped_Competition)/urdf/obstacles/Component_7__189942_.urdf.xacro"/>
+	<!-- Component_7__189945_ -->
+	<xacro:include filename="$(find ICRA2023_Quadruped_Competition)/urdf/obstacles/Component_7__189945_.urdf.xacro"/>
+	<!-- Component_7__189948_ -->
+	<xacro:include filename="$(find ICRA2023_Quadruped_Competition)/urdf/obstacles/Component_7__189948_.urdf.xacro"/>
+	<!-- Component_7__189951_ -->
+	<xacro:include filename="$(find ICRA2023_Quadruped_Competition)/urdf/obstacles/Component_7__189951_.urdf.xacro"/>
+	<!-- Component_7__189954_ -->
+	<xacro:include filename="$(find ICRA2023_Quadruped_Competition)/urdf/obstacles/Component_7__189954_.urdf.xacro"/>
+	<!-- Component_7__189957_ -->
+	<xacro:include filename="$(find ICRA2023_Quadruped_Competition)/urdf/obstacles/Component_7__189957_.urdf.xacro"/>
+	<!-- Component_7__189960_ -->
+	<xacro:include filename="$(find ICRA2023_Quadruped_Competition)/urdf/obstacles/Component_7__189960_.urdf.xacro"/>
+	<!-- Component_7__189963_ -->
+	<xacro:include filename="$(find ICRA2023_Quadruped_Competition)/urdf/obstacles/Component_7__189963_.urdf.xacro"/>
+	<!-- Component_7__189966_ -->
+	<xacro:include filename="$(find ICRA2023_Quadruped_Competition)/urdf/obstacles/Component_7__189966_.urdf.xacro"/>
+	<!-- Component_7__189969_ -->
+	<xacro:include filename="$(find ICRA2023_Quadruped_Competition)/urdf/obstacles/Component_7__189969_.urdf.xacro"/>
+	<!-- Component_7__189972_ -->
+	<xacro:include filename="$(find ICRA2023_Quadruped_Competition)/urdf/obstacles/Component_7__189972_.urdf.xacro"/>
+	<!-- Component_7__189975_ -->
+	<xacro:include filename="$(find ICRA2023_Quadruped_Competition)/urdf/obstacles/Component_7__189975_.urdf.xacro"/>
+	<!-- Component_7__189978_ -->
+	<xacro:include filename="$(find ICRA2023_Quadruped_Competition)/urdf/obstacles/Component_7__189978_.urdf.xacro"/>
+	<!-- Component_7__189981_ -->
+	<xacro:include filename="$(find ICRA2023_Quadruped_Competition)/urdf/obstacles/Component_7__189981_.urdf.xacro"/>
+	<!-- Component_7__189984_ -->
+	<xacro:include filename="$(find ICRA2023_Quadruped_Competition)/urdf/obstacles/Component_7__189984_.urdf.xacro"/>
+	<!-- Component_7__189987_ -->
+	<xacro:include filename="$(find ICRA2023_Quadruped_Competition)/urdf/obstacles/Component_7__189987_.urdf.xacro"/>
+	<!-- Component_7__189990_ -->
+	<xacro:include filename="$(find ICRA2023_Quadruped_Competition)/urdf/obstacles/Component_7__189990_.urdf.xacro"/>
+	<!-- Component_7__190005_ -->
+	<xacro:include filename="$(find ICRA2023_Quadruped_Competition)/urdf/obstacles/Component_7__190005_.urdf.xacro"/>
+	<!-- Component_7__190008_ -->
+	<xacro:include filename="$(find ICRA2023_Quadruped_Competition)/urdf/obstacles/Component_7__190008_.urdf.xacro"/>
+	<!-- Component_7__190011_ -->
+	<xacro:include filename="$(find ICRA2023_Quadruped_Competition)/urdf/obstacles/Component_7__190011_.urdf.xacro"/>
+	<!-- Component_7__190014_ -->
+	<xacro:include filename="$(find ICRA2023_Quadruped_Competition)/urdf/obstacles/Component_7__190014_.urdf.xacro"/>
+	<!-- Component_7__190017_ -->
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