Commit message: add: urdf.xacro

File: urdf/obstacles/Component_7__190053_.urdf.xacro (robot description, xacro)
@@ -1,11 +1,11 @@
 <?xml version="1.0" encoding="utf-8"?>
-<robot xmlns:xacro="http://www.ros.org/wiki/xacro">
-	<xacro:macro name="obj_1200x2400_OSB" params="handle parent position orientation">
-	<joint name="1200x2400_OSB${handle}_joint" type="fixed">
+<robot xmlns:xacro="http://ros.org/wiki/xacro">
+	<xacro:macro name="obs_Component_7__190053_" params="handle parent position orientation">
+	<joint name="Component_7__190053_${handle}_joint" type="fixed">
 		<origin xyz="${position}" rpy="${orientation}"/>
 		<parent link="${parent}"/>
-		<child link="1200x2400_OSB${handle}"/>
+		<child link="Component_7__190053_${handle}"/>
 	</joint>
-	<link name="1200x2400_OSB${handle}">
+	<link name="Component_7__190053_${handle}">
 		<inertial>
 			<origin xyz="0 0 0" rpy="0 0 0"/>
@@ -19,5 +19,5 @@
 			<origin xyz="0 0 0" rpy="0 0 0"/>
 			<geometry>
-				<mesh filename="package://ICRA2023_Quadruped_Competition/meshes/assembly/1200x2400_OSB.obj"/>
+				<mesh filename="package://ICRA2023_Quadruped_Competition/meshes/assembly/Component_7__190053_.obj"/>
 			</geometry>
 			<material name="">
@@ -27,5 +27,5 @@
 			<origin xyz="0 0 0" rpy="0 0 0"/>
 			<geometry>
-				<mesh filename="package://ICRA2023_Quadruped_Competition/meshes/assembly/1200x2400_OSB.obj"/>
+				<mesh filename="package://ICRA2023_Quadruped_Competition/meshes/assembly/Component_7__190053_.obj"/>
 			</geometry>
 			<material name="">
@@ -33,5 +33,5 @@
 		</collision>
 	</link>
-	<gazebo reference="1200x2400_OSB${handle}">
+	<gazebo reference="Component_7__190053_${handle}">
 	</gazebo>
 	</xacro:macro>

Commit message: update: map level

File: urdf/map.urdf.xacro (robot description, xacro)
@@ -1,7 +1,8 @@
 <?xml version="1.0" ?>
 <robot xmlns:xacro="http://ros.org/wiki/xacro" name="competition_map">
+ 	<xacro:arg name="course" default="part"/>
 	<link name="world"/>
 	<xacro:include filename="$(find ICRA2023_Quadruped_Competition)/urdf/maps/map_part.urdf.xacro"/>
-	<xacro:map_part parent="world" handle="1" position="0 0 0" orientation="0.0 0.0 0.0"/>
+	<xacro:map_part parent="world" handle="1" position="0 0 0" orientation="0.0 0.0 0.0" course="$(arg course)"/>
 	<gazebo>
 		<static>true</static>

File: urdf/maps/map_part.urdf.xacro (robot description, xacro)
@@ -1,5 +1,5 @@
 <?xml version="1.0" encoding="utf-8"?>
 <robot xmlns:xacro="http://www.ros.org/wiki/xacro">
-  <xacro:macro name="map_part" params="handle parent position orientation">
+  <xacro:macro name="map_part" params="handle parent position orientation course">
   <joint name="map_part${handle}_joint" type="fixed">
     <origin xyz="${position}" rpy="${orientation}"/>
@@ -23,5 +23,5 @@
         <geometry>
           <mesh
-            filename="package://ICRA2023_Quadruped_Competition/meshes/part/map_part.dae"/>
+            filename="package://ICRA2023_Quadruped_Competition/meshes/part/map_${course}.dae"/>
         </geometry>
         <material name="">
@@ -35,5 +35,5 @@
         <geometry>
           <mesh
-            filename="package://ICRA2023_Quadruped_Competition/meshes/part/map_part.dae"/>
+            filename="package://ICRA2023_Quadruped_Competition/meshes/part/map_${course}.dae"/>
         </geometry>
         <material name="">
